File: kicad/bike-sensors-redbear-duo.sch (KiCad schematic (older format))
At the start: 4 parts

Commit message: Continued work on the schematic and starting to understand how the footprint works.
Parts:
- added C8: 220u, symbol CP1
- added Q4: P_Channel_MOSFET, symbol P_Channel_MOSFET
- added R6: R20K, symbol R
- added R7: R10K, symbol R
- added R9: R150, symbol R
- gave numbers to parts that had none: 4
Connections:
- net at TH1.1 (VDD): now also U2.12 (3V3), U3.6 (Vcc), U5.4 (Vc), U5.6 (Vc), R9.2
- net at TH1.2 (DATA): now also U2.7 (D6), R7.2
- net GND: now reaches TH1.4 (GND)
- net GND: now also U2.14 (GND), U3.2 (LED-GND), U3.4 (S-GND), U5.5 (Vh-), C8.2, R6.2
- net at U3.1 (V-LED): now also C8.1, R9.1
- net at U3.3 (LED): now also U2.24 (A0)
- net at U3.5 (Vo): now also U2.22 (A2)
- net at U5.1 (Vrl): now also U2.20 (A4), U5.3 (Vrl)
- net at U5.2 (Vh): now also Q4.2 (Drain)
- net at U2.13 (VIN): now also Q4.3 (Source)
- net at U2.4 (D3): now also Q4.1 (Gate)
Other:
- moved on the sheet: U2, U3, U5
Changed lines of the file:
@@
 $EndDescr
 $Comp
-L DHT22_Temperature_Humidity TH?
+L DHT22_Temperature_Humidity TH1
 U 1 1 576E2AD2
 P 2250 2300
-F 0 "TH?" H 2250 3350 60  0000 C CNN
+F 0 "TH1" H 2250 3350 60  0000 C CNN
 F 1 "DHT22_Temperature_Humidity" H 2250 3250 60  0000 C CNN
 F 2 "" H 2250 2300 60  0000 C CNN
@@
 $EndComp
 $Comp
-L GP2Y10_Dust_Particulate U?
+L GP2Y10_Dust_Particulate U3
 U 1 1 576E3133
-P 8250 1700
-F 0 "U?" H 8100 1800 60  0000 C CNN
-F 1 "GP2Y10_Dust_Particulate" H 8100 1700 60  0000 C CNN
-F 2 "" H 8100 1700 60  0000 C CNN
-F 3 "" H 8100 1700 60  0000 C CNN
-	1    8250 1700
-	1    0    0    -1
-$EndComp
-$Comp
-L MQ-7_Carbon_Monoxide U?
+P 6900 1550
+F 0 "U3" H 6750 1650 60  0000 C CNN
+F 1 "GP2Y10_Dust_Particulate" H 6750 1550 60  0000 C CNN
+F 2 "" H 6750 1550 60  0000 C CNN
+F 3 "" H 6750 1550 60  0000 C CNN
+	1    6900 1550
+	1    0    0    -1
+$EndComp
+$Comp
+L MQ-7_Carbon_Monoxide U5
 U 1 1 576E32E5
-P 7550 3700
-F 0 "U?" H 7550 3700 60  0000 C CNN
-F 1 "MQ-7_Carbon_Monoxide" H 7550 3600 60  0000 C CNN
-F 2 "" H 7550 3700 60  0000 C CNN
-F 3 "" H 7550 3700 60  0000 C CNN
-	1    7550 3700
-	1    0    0    -1
-$EndComp
-$Comp
-L Redbear_Duo U?
+P 7550 5450
+F 0 "U5" H 7550 5450 60  0000 C CNN
+F 1 "MQ-7_Carbon_Monoxide" H 7550 5350 60  0000 C CNN
+F 2 "" H 7550 5450 60  0000 C CNN
+F 3 "" H 7550 5450 60  0000 C CNN
+	1    7550 5450
+	1    0    0    -1
+$EndComp
+$Comp
+L Redbear_Duo U2
 U 1 1 576E35B2
-P 4300 2500
-F 0 "U?" H 4900 2650 60  0000 C CNN
-F 1 "Redbear_Duo" H 4900 2550 60  0000 C CNN
-F 2 "" H 4300 2500 60  0000 C CNN
-F 3 "" H 4300 2500 60  0000 C CNN
-	1    4300 2500
-	1    0    0    -1
-$EndComp
+P 3500 3900
+F 0 "U2" H 4100 4050 60  0000 C CNN
+F 1 "Redbear_Duo" H 4100 3950 60  0000 C CNN
+F 2 "" H 3500 3900 60  0000 C CNN
+F 3 "" H 3500 3900 60  0000 C CNN
+	1    3500 3900
+	1    0    0    -1
+$EndComp
+$Comp
+L CP1 C8
+U 1 1 57738F5C
+P 6050 3200
+F 0 "C8" H 6075 3300 50  0000 L CNN
+F 1 "220u" H 6075 3100 50  0000 L CNN
+F 2 "" H 6050 3200 50  0000 C CNN
+F 3 "" H 6050 3200 50  0000 C CNN
+	1    6050 3200
+	0    -1   -1   0
+$EndComp
+Wire Wire Line
+	6100 2500 6100 2600
+Wire Wire Line
+	6100 2600 5900 2600
+Wire Wire Line
+	5900 2600 5900 3200
+Connection ~ 6200 3200
+Wire Wire Line
+	6600 2500 6600 5400
+Wire Wire Line
+	3600 5400 7900 5400
+Wire Wire Line
+	3600 5400 3600 5200
+$Comp
+L R R9
+U 1 1 577393B5
+P 6450 2800
+F 0 "R9" V 6530 2800 50  0000 C CNN
+F 1 "R150" V 6450 2800 50  0000 C CNN
+F 2 "" V 6380 2800 50  0000 C CNN
+F 3 "" H 6450 2800 50  0000 C CNN
+	1    6450 2800
+	0    -1   -1   0
+$EndComp
+Connection ~ 6600 2800
+Wire Wire Line
+	6300 2800 5900 2800
+Connection ~ 5900 2800
+Wire Wire Line
+	6300 2500 6300 4100
+Wire Wire Line
+	6300 4100 4600 4100
+Wire Wire Line
+	6500 2500 6500 4300
+Wire Wire Line
+	6500 4300 4600 4300
+Wire Wire Line
+	2100 2300 2100 5200
+Wire Wire Line
+	2100 5200 3600 5200
+$Comp
+L R R7
+U 1 1 5773ACC3
+P 2250 2700
+F 0 "R7" V 2330 2700 50  0000 C CNN
+F 1 "R10K" V 2250 2700 50  0000 C CNN
+F 2 "" V 2180 2700 50  0000 C CNN
+F 3 "" H 2250 2700 50  0000 C CNN
+	1    2250 2700
+	0    -1   -1   0
+$EndComp
+Wire Wire Line
+	2200 2300 2200 2500
+Wire Wire Line
+	2200 2500 2400 2500
+Wire Wire Line
+	2400 2500 2400 4700
+Wire Wire Line
+	2400 4700 3600 4700
+Connection ~ 2400 2700
+$Comp
+L P_Channel_MOSFET Q4
+U 1 1 5773B3DF
+P 8100 2900
+F 0 "Q4" H 8100 3000 60  0000 C CNN
+F 1 "P_Channel_MOSFET" H 8100 2900 60  0000 C CNN
+F 2 "" H 8100 2900 60  0000 C CNN
+F 3 "" H 8100 2900 60  0000 C CNN
+	1    8100 2900
+	1    0    0    -1
+$EndComp
+$Comp
+L GND #PWR?
+U 1 1 57774C81
+P 2600 2300
+F 0 "#PWR?" H 2600 2050 50  0001 C CNN
+F 1 "GND" H 2600 2150 50  0000 C CNN
+F 2 "" H 2600 2300 50  0000 C CNN
+F 3 "" H 2600 2300 50  0000 C CNN
+	1    2600 2300
+	1    0    0    -1
+$EndComp
+Wire Wire Line
+	2400 2300 2600 2300
+Wire Wire Line
+	6200 2500 6200 3500
+Wire Wire Line
+	6400 3500 6400 2500
+Wire Wire Line
+	5600 3500 6400 3500
+$Comp
+L GND #PWR?
+U 1 1 57774DFC
+P 5600 3500
+F 0 "#PWR?" H 5600 3250 50  0001 C CNN
+F 1 "GND" H 5600 3350 50  0000 C CNN
+F 2 "" H 5600 3500 50  0000 C CNN
+F 3 "" H 5600 3500 50  0000 C CNN
+	1    5600 3500
+	1    0    0    -1
+$EndComp
+Connection ~ 6200 3500
+$Comp
+L GND #PWR?
+U 1 1 57774E44
+P 5000 5600
+F 0 "#PWR?" H 5000 5350 50  0001 C CNN
+F 1 "GND" H 5000 5450 50  0000 C CNN
+F 2 "" H 5000 5600 50  0000 C CNN
+F 3 "" H 5000 5600 50  0000 C CNN
+	1    5000 5600
+	1    0    0    -1
+$EndComp
+Wire Wire Line
+	4600 5100 5000 5100
+Wire Wire Line
+	5000 4800 5000 5600
+Wire Wire Line
+	8000 3800 3500 3800
+Wire Wire Line
+	3500 3800 3500 4400
+Wire Wire Line
+	3500 4400 3600 4400
+Wire Wire Line
+	8200 3800 8200 5200
+Wire Wire Line
+	8200 5200 4600 5200
+Wire Wire Line
+	8100 3800 8100 5100
+Wire Wire Line
+	8100 5100 6800 5100
+Wire Wire Line
+	6800 5100 6800 5900
+Wire Wire Line
+	6800 5900 7150 5900
+$Comp
+L GND #PWR?
+U 1 1 57775BB9
+P 8500 5900
+F 0 "#PWR?" H 8500 5650 50  0001 C CNN
+F 1 "GND" H 8500 5750 50  0000 C CNN
+F 2 "" H 8500 5900 50  0000 C CNN
+F 3 "" H 8500 5900 50  0000 C CNN
+	1    8500 5900
+	1    0    0    -1
+$EndComp
+Wire Wire Line
+	7950 5900 8500 5900
+Wire Wire Line
+	7200 6050 7200 5750
+Wire Wire Line
+	7200 5750 6000 5750
+Wire Wire Line
+	6000 5750 6000 4500
+Wire Wire Line
+	6000 4500 4600 4500
+$Comp
+L R R6
+U 1 1 57775D75
+P 5000 4650
+F 0 "R6" V 5080 4650 50  0000 C CNN
+F 1 "R20K" V 5000 4650 50  0000 C CNN
+F 2 "" V 4930 4650 50  0000 C CNN
+F 3 "" H 5000 4650 50  0000 C CNN
+	1    5000 4650
+	1    0    0    -1
+$EndComp
+Connection ~ 5000 5100
+Wire Wire Line
+	7900 5400 7900 6050
+Connection ~ 7900 5750
+Connection ~ 6600 5400
 $EndSCHEMATC

Commit message: Fixed the resistor junctions.
Connections:
- net at R9.2, TH1.1 (VDD), U2.12 (3V3)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: now also R7.1
- net at U2.20 (A4), U5.1 (Vrl), U5.3 (Vrl): now also R6.1
Changed lines of the file:
@@
 $EndComp
 $Comp
-L GND #PWR?
+L GND #PWR01
 U 1 1 57774C81
 P 2600 2300
-F 0 "#PWR?" H 2600 2050 50  0001 C CNN
+F 0 "#PWR01" H 2600 2050 50  0001 C CNN
 F 1 "GND" H 2600 2150 50  0000 C CNN
 F 2 "" H 2600 2300 50  0000 C CNN
@@
 	5600 3500 6400 3500
 $Comp
-L GND #PWR?
+L GND #PWR02
 U 1 1 57774DFC
 P 5600 3500
-F 0 "#PWR?" H 5600 3250 50  0001 C CNN
+F 0 "#PWR02" H 5600 3250 50  0001 C CNN
 F 1 "GND" H 5600 3350 50  0000 C CNN
 F 2 "" H 5600 3500 50  0000 C CNN
@@
 Connection ~ 6200 3500
 $Comp
-L GND #PWR?
+L GND #PWR03
 U 1 1 57774E44
 P 5000 5600
-F 0 "#PWR?" H 5000 5350 50  0001 C CNN
+F 0 "#PWR03" H 5000 5350 50  0001 C CNN
 F 1 "GND" H 5000 5450 50  0000 C CNN
 F 2 "" H 5000 5600 50  0000 C CNN
@@
 	6800 5900 7150 5900
 $Comp
-L GND #PWR?
+L GND #PWR04
 U 1 1 57775BB9
 P 8500 5900
-F 0 "#PWR?" H 8500 5650 50  0001 C CNN
+F 0 "#PWR04" H 8500 5650 50  0001 C CNN
 F 1 "GND" H 8500 5750 50  0000 C CNN
 F 2 "" H 8500 5900 50  0000 C CNN
@@
 Connection ~ 7900 5750
 Connection ~ 6600 5400
+Connection ~ 2100 2700
+Connection ~ 5000 4500
 $EndSCHEMATC
